File: hardware/Accessories/Etch-A-Sketch Controller/etch-a-sketch.sch (KiCad schematic (older format))
At the start: 27 parts

Commit message: Add power flags
Parts:
- gave numbers to parts that had none: 27
Connections:
- wire segments 78 -> 80
