File: hardware/Accessories/Etch-A-Sketch Controller/etch-a-sketch.sch (KiCad schematic (older format))
At the start: 27 parts, among them SW1 DPST, SW2 DPST, SW3 DPST, SW4 DPST

Commit message: Add encoder with gnd shield connection.
Parts:
- removed EN1, EN2: MISC_ENCODER_5_PINS, ~, symbol MISC_ENCODER_5_PINS
- added EN1, EN2: ENCODER_5_PINS, ~, symbol MISC_ENCODER_5_PINS_W_SHIELD
Connections:
- wire segments 80 -> 82
Changed lines of the file:
@@
 Sheet 1 1
 Title "Etch-a-Sketch"
-Date "26 mar 2015"
+Date "30 mar 2015"
 Rev "1.0"
 Comp "BQ"
@@
 	1    3600 4850
 	1    0    0    -1
-$EndComp
-$Comp
-L MISC_ENCODER_5_PINS EN1
-U 1 1 5512B2F8
-P 1450 1750
-F 0 "EN1" H 1600 2050 60  0000 C CNN
-F 1 "MISC_ENCODER_5_PINS" H 1450 1450 60  0000 C CNN
-F 2 "~" H 1450 1750 60  0000 C CNN
-F 3 "~" H 1450 1750 60  0000 C CNN
-	1    1450 1750
-	-1   0    0    -1
 $EndComp
 $Comp
@@
 	2150 1750 2150 1850
 Wire Wire Line
-	950  1650 750  1650
+	950  1600 750  1600
 $Comp
 L GND #PWR06
 U 1 1 5512B5F3
-P 850 1950
-F 0 "#PWR06" H 850 1950 30  0001 C CNN
-F 1 "GND" H 850 1880 30  0001 C CNN
-F 2 "" H 850 1950 60  0000 C CNN
-F 3 "" H 850 1950 60  0000 C CNN
-	1    850  1950
-	-1   0    0    -1
-$EndComp
-Wire Wire Line
-	850  1850 850  1950
-Wire Wire Line
-	850  1850 950  1850
-Text Label 750  1650 0    60   ~ 0
+P 850 2150
+F 0 "#PWR06" H 850 2150 30  0001 C CNN
+F 1 "GND" H 850 2080 30  0001 C CNN
+F 2 "" H 850 2150 60  0000 C CNN
+F 3 "" H 850 2150 60  0000 C CNN
+	1    850  2150
+	-1   0    0    -1
+$EndComp
+Wire Wire Line
+	850  1800 850  2150
+Wire Wire Line
+	850  1800 950  1800
+Text Label 750  1600 0    60   ~ 0
 D2
 Text Label 3050 1350 2    60   ~ 0
@@
 Text Label 3050 2150 2    60   ~ 0
 D0
-$Comp
-L MISC_ENCODER_5_PINS EN2
-U 1 1 5512B615
-P 4250 1750
-F 0 "EN2" H 4400 2050 60  0000 C CNN
-F 1 "MISC_ENCODER_5_PINS" H 4250 1450 60  0000 C CNN
-F 2 "~" H 4250 1750 60  0000 C CNN
-F 3 "~" H 4250 1750 60  0000 C CNN
-	1    4250 1750
-	-1   0    0    -1
-$EndComp
 $Comp
 L C C4
@@
 	4950 1750 4950 1850
 Wire Wire Line
-	3750 1650 3550 1650
+	3750 1600 3550 1600
 $Comp
 L GND #PWR012
 U 1 1 5512B676
-P 3650 1950
-F 0 "#PWR012" H 3650 1950 30  0001 C CNN
-F 1 "GND" H 3650 1880 30  0001 C CNN
-F 2 "" H 3650 1950 60  0000 C CNN
-F 3 "" H 3650 1950 60  0000 C CNN
-	1    3650 1950
-	-1   0    0    -1
-$EndComp
-Wire Wire Line
-	3650 1850 3650 1950
-Wire Wire Line
-	3650 1850 3750 1850
-Text Label 3550 1650 0    60   ~ 0
+P 3600 2150
+F 0 "#PWR012" H 3600 2150 30  0001 C CNN
+F 1 "GND" H 3600 2080 30  0001 C CNN
+F 2 "" H 3600 2150 60  0000 C CNN
+F 3 "" H 3600 2150 60  0000 C CNN
+	1    3600 2150
+	-1   0    0    -1
+$EndComp
+Wire Wire Line
+	3600 1800 3600 2150
+Wire Wire Line
+	3600 1800 3750 1800
+Text Label 3550 1600 0    60   ~ 0
 D21
 Text Label 5850 1350 2    60   ~ 0
@@
 Wire Wire Line
 	1150 7300 1150 7400
+$Comp
+L MISC_ENCODER_5_PINS_W_SHIELD EN1
+U 1 1 55192834
+P 1450 1750
+F 0 "EN1" H 1600 2050 60  0000 C CNN
+F 1 "ENCODER_5_PINS" H 1450 1450 60  0000 C CNN
+F 2 "~" H 1450 1750 60  0000 C CNN
+F 3 "~" H 1450 1750 60  0000 C CNN
+	1    1450 1750
+	-1   0    0    -1
+$EndComp
+Wire Wire Line
+	850  1900 950  1900
+Connection ~ 850  1900
+$Comp
+L MISC_ENCODER_5_PINS_W_SHIELD EN2
+U 1 1 551928D0
+P 4250 1750
+F 0 "EN2" H 4400 2050 60  0000 C CNN
+F 1 "ENCODER_5_PINS" H 4250 1450 60  0000 C CNN
+F 2 "~" H 4250 1750 60  0000 C CNN
+F 3 "~" H 4250 1750 60  0000 C CNN
+	1    4250 1750
+	-1   0    0    -1
+$EndComp
+Wire Wire Line
+	3750 1900 3600 1900
+Connection ~ 3600 1900
 $EndSCHEMATC
