File: hardware/Accessories/Etch-A-Sketch Controller/etch-a-sketch.kicad_pcb (KiCad board)
At the start: 2 copper layers, 98 x 75 mm, 31 parts, among them SW1 DPST, SW2 DPST, SW3 DPST, SW4 DPST

Commit message: Add encoder with gnd shield connection.
Parts:
- EN1, EN2: value MISC_ENCODER_5_PINS -> ENCODER_5_PINS; footprint MISC_ENCODER_5_PINS -> Misc_Encoder_5_Pins_w_shield
- moved EN2 0.13 mm to (186.9, 84.2)
